File: kicad/Interface.kicad_sch (KiCad schematic)
At the start: 13 parts, among them J2 DBG-TGT, U10 USB6B1, U7 74AUP1G17, U8 74AUP1G17, U9 USB6B1

Commit message: starting redesign
Parts:
- added R16, R17, R18: 100, Resistor_SMD:R_0603_1608Metric, symbol Device:R
Connections:
- net GND: no longer J2.2 (Pin_2)
- net UART0_TX: now also R17.1; no longer U10.2 (I/O1)
- net UART1_TX: now also R16.1; no longer U9.2 (I/O1)
- new net RESET: J2.2 (Pin_2), R18.2
- new net SWCLK: R17.2, U10.2 (I/O1)
- new net TGT_RST: R18.1
- new net UART_TX: R16.2, U9.2 (I/O1)
Other:
- moved on the sheet: R13, R14
