File: kicad/RP2040.kicad_sch (KiCad schematic)
At the start: 31 parts, among them SW1 SW_Push, U5 RP2040, U6 W25Q16JVSS, Y1 12MHz

Commit message: starting redesign
Parts:
- R5, R6: value 1k -> 22; LCSC C21190 -> C1203; MPN_LCSC 0603WAF1001T5E -> 0603WAJ0220T5E
Connections:
- net TGT_RST: now reaches U5.3 (GPIO1)
Changed lines of the file:
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@@
 	(wire
 		(pts
+			(xy 177.8 76.2) (xy 194.31 76.2)
+		)
+		(stroke
+			(width 0)
+			(type default)
+		)
+	)
+	(wire
+		(pts
 			(xy 99.06 41.91) (xy 99.06 45.72)
 		)
@@
 		)
 	)
+	(hierarchical_label "TGT_RST"
+		(shape output)
+		(at 194.31 76.2 0)
+		(effects
+			(font
+				(size 1.27 1.27)
+			)
+			(justify left)
+		)
+	)
 	(symbol
 		(lib_id "Device:C")
@@
 			)
 		)
-		(property "Value" "1k"
+		(property "Value" "22"
 			(at 102.87 99.06 90)
 			(effects
@@
 			)
 		)
-		(property "LCSC" "C21190"
+		(property "LCSC" "C1203"
 			(at 102.87 99.06 90)
 			(effects
@@
 			)
 		)
-		(property "MPN_LCSC" "0603WAF1001T5E"
+		(property "MPN_LCSC" "0603WAJ0220T5E"
 			(at 102.87 99.06 90)
 			(effects
@@
 			)
 		)
-		(property "Value" "1k"
+		(property "Value" "22"
 			(at 102.87 96.52 90)
 			(effects
@@
 			)
 		)
-		(property "LCSC" "C21190"
+		(property "LCSC" "C1203"
 			(at 102.87 96.52 90)
 			(effects
@@
 			)
 		)
-		(property "MPN_LCSC" "0603WAF1001T5E"
+		(property "MPN_LCSC" "0603WAJ0220T5E"
 			(at 102.87 96.52 90)
 			(effects
