File: kicad/USB_input_isolation.kicad_sch (KiCad schematic)
At the start: 19 parts, among them J1 USB_C_Receptacle_USB2.0_14P, U2 ADUM3160, U3 USB6B1, U4 NCP1117-3.3_SOT223

Commit message: starting redesign
Parts:
- added C27: 10u, Capacitor_SMD:C_0805_2012Metric, symbol Device:C
- added FB1: ~, symbol Device:FerriteBead_Small
- added L1: 744232090, Inductor_SMD:L_CommonMode_Wurth_WE-CNSW-1206, symbol Filter:Choke_Wurth_WE-CNSW_744232090
Connections:
- net GNDPWR: now also C27.2
- net UD+: now also L1.3; no longer U3.6 (I/O2)
- net UD-: now also L1.2; no longer U3.7 (I/O1)
- net at C1.1, C2.1, C25.1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: now also FB1.2; no longer F1.2, U3.1 (VBUS), U3.8 (VBUS)
- new net: C27.1, F1.2, FB1.1, U3.1 (VBUS), U3.8 (VBUS)
- new net: L1.4, U3.6 (I/O2)
- new net: L1.1, U3.7 (I/O1)
Other:
- note added: "!! Y-Class capacitor !!"
- note added: "5V/500mA"
- note added: "7.4 kHz PI-Filter"
- note added: "Keep filters and ESD protection on separate GND island!"
- note added: "USB Common Mode Choke"
- moved on the sheet: C1, F1, J1, R1, R2, U3
