File: kicad/isolated_rp2040_debugger.kicad_pcb (KiCad board)
At the start: 4 copper layers, 91 x 44 mm, 67 parts, among them J1 USB_C_Receptacle_USB2.0_14P, J2 DBG-TGT, SW1 SW_Push, U10 USB6B1, U2 ADUM3160, U3 USB6B1, U4 NCP1117-3.3_SOT223, U5 RP2040, U6 W25Q16JVSS, U7 74AUP1G17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

Commit message: starting redesign
Parts:
- added C27: 10u, Capacitor_SMD:C_0805_2012Metric, F.Cu at (64.5, 89.0)
- added FB1: ~, Inductor_SMD:L_0805_2012Metric, F.Cu at (64.5, 91.0)
- added L1: 744232090, Inductor_SMD:L_CommonMode_Wurth_WE-CNSW-1206, F.Cu at (70.5, 99.5)
- added R16: 100, Resistor_SMD:R_0603_1608Metric, F.Cu at (98.4, 57.8)
- added R17: 100, Resistor_SMD:R_0603_1608Metric, F.Cu at (98.4, 60.3)
- added R18: 100, Resistor_SMD:R_0603_1608Metric, F.Cu at (98.4, 62.8)
- R5, R6: value 1k -> 22
- moved C2 45.8 mm to (53.9, 137.1)
- moved C25 29.2 mm to (94.8, 129.5)
- moved C26 29.2 mm to (106.0, 129.5)
- moved C5 29.2 mm to (93.3, 133.5)
- moved C6 29.2 mm to (107.3, 133.5)
- moved C9 28.3 mm to (78.5, 130.0)
- moved U2 15.8 mm to (80.0, 98.0)
- moved R2 7.55 mm to (60.5, 102.0)
- moved C1 6.15 mm to (64.5, 93.0)
- moved R1 4.62 mm to (60.5, 103.5)
- moved F1 4.57 mm to (60.0, 94.0)
- moved U3 4.47 mm to (63.0, 98.0)
- moved U1 4.38 mm to (80.5, 84.5)
- moved C10 4.23 mm to (109.2, 102.8)
- moved C11 4.23 mm to (114.2, 102.8)
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Connections:
- net /RP2040/USB_D+ renamed /Galvanic Isolation/USB_D+
- net /RP2040/USB_D- renamed /Galvanic Isolation/USB_D-
- net /USB Input Isolation/UDC+ renamed /USB Input Protection & Filter/UDC+
- net /USB Input Isolation/UDC- renamed /USB Input Protection & Filter/UDC-
- C1 pad 1: Net-(U1-Vin+) -> +5V
- C2 pad 1: Net-(U1-Vin+) -> +5V
- C25 pad 1: Net-(U1-Vin+) -> +5V
- C3 pad 1: +5V -> Net-(U1-Vout+)
- C4 pad 1: +5V -> Net-(U1-Vout+)
- C7 pad 1: +5V -> Net-(U1-Vout+)
- F1 pad 2: Net-(U1-Vin+) -> Net-(C27-Pad1)
- J2 pad 2: GND -> /Interface/RESET
- U1 pad 2: Net-(U1-Vin+) -> +5V
- U1 pad 8: +5V -> Net-(U1-Vout+)
- U2 pad 1: Net-(U1-Vin+) -> +5V
- U2 pad 6: /USB Input Isolation/UD- -> /Galvanic Isolation/USB_HOST_D-
- U2 pad 7: /USB Input Isolation/UD+ -> /Galvanic Isolation/USB_HOST_D+
- U3 pad 1: Net-(U1-Vin+) -> Net-(C27-Pad1)
- U3 pad 6: /USB Input Isolation/UD+ -> /USB Input Protection & Filter/DF+
- U3 pad 7: /USB Input Isolation/UD- -> /USB Input Protection & Filter/DF-
- U3 pad 8: Net-(U1-Vin+) -> Net-(C27-Pad1)
- U4 pad 3: +5V -> Net-(U1-Vout+)
- U5 pad 15: /Interface/SWCLK -> /Interface/UART0_TX
- U5 pad 3: unconnected-(U5-GPIO1-Pad3) -> /RP2040/TGT_RST
- U5 pad 6: /Interface/UART_TX -> /Interface/UART1_TX
Routing:
- net GND: track 471.0 -> 0.00 mm, vias 155 -> 0
- net GNDPWR: track 290.9 -> 5.34 mm, vias 76 -> 61
- net +3V3: track 224.7 -> 0.00 mm, vias 11 -> 0
- net /Interface/UART1_RX: track 49.6 -> 0.00 mm, vias 2 -> 0
- net /Interface/UART_TX: track 45.3 -> 0.00 mm, vias 2 -> 0
- net /Interface/GPIO6: track 42.9 -> 0.00 mm, vias 2 -> 0
- net +1V1: track 41.5 -> 0.00 mm, vias 7 -> 0
- net Net-(U1-Vin+): track 38.8 -> 0.00 mm
- net /Interface/UART0_RX: track 33.9 -> 0.00 mm, vias 2 -> 0
- net Net-(U5-GPIO2): track 28.8 -> 0.00 mm, vias 2 -> 0
- net Net-(J2-Pin_1): track 28.6 -> 0.00 mm
- net /Interface/GPIO14: track 26.7 -> 0.00 mm, vias 2 -> 0
- net /Interface/SWCLK: track 23.3 -> 0.00 mm, vias 2 -> 0
- net /USB Input Isolation/UD-: track 23.0 -> 0.00 mm
- net /USB Input Isolation/UD+: track 23.0 -> 0.00 mm
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- added copper zone on B.Cu, net GNDPWR
- added copper zone on F.Cu, net GNDPWR
- removed copper zone on F.Cu, net +3V3
- removed copper zone on F.Cu, net +5V
- removed copper zone on F.Cu, net GND
- removed copper zone on In1.Cu, net GND
- removed copper zone on In2.Cu, net GND
Other:
- board size 91 x 44 mm -> 108 x 51.5 mm
- board text removed: "+3V3"
- board text removed: "Based on Raspberry Pi Probe Design Schematics 2026 Peter Heinrich REV: A"
- board text removed: "CLK"
- board text removed: "CON"
- board text removed: "DIO"
- board text removed: "Enclosure: CU-1872-B"
- board text removed: "GND"
- board text removed: "Isolated Debug Probe"
- board text removed: "PC GND"
- board text removed: "PWR"
- board text removed: "RUN"
- board text removed: "RX"
- board text removed: "TARGET GND"
- board text removed: "TARGET POWER"
- board text removed: "TX"
