File: kicad/isolated_rp2040_debugger.kicad_sch (KiCad schematic)
At the start: 4 parts

Commit message: starting redesign
Other:
- sheet USB Input Isolation renamed USB Input Protection & Filter
- added sheet Galvanic Isolation (galvanic_isolation.kicad_sch)
- sheet RP2040 ports: added TGT_RST; removed none
- sheet USB Input Protection & Filter: file USB_input_isolation.kicad_sch -> USB_input_protection.kicad_sch
- sheet USB Input Protection & Filter ports: added USB_HOST_D+, USB_HOST_D-; removed USB_D+, USB_D-
Changed lines of the file:
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@@
 	(wire
 		(pts
-			(xy 113.03 64.77) (xy 119.38 64.77)
-		)
-		(stroke
-			(width 0)
-			(type default)
-		)
-	)
-	(wire
-		(pts
-			(xy 113.03 80.01) (xy 119.38 80.01)
-		)
-		(stroke
-			(width 0)
-			(type default)
-		)
-	)
-	(wire
-		(pts
-			(xy 113.03 69.85) (xy 119.38 69.85)
-		)
-		(stroke
-			(width 0)
-			(type default)
-		)
-	)
-	(wire
-		(pts
-			(xy 113.03 67.31) (xy 119.38 67.31)
-		)
-		(stroke
-			(width 0)
-			(type default)
-		)
-	)
-	(wire
-		(pts
-			(xy 73.66 64.77) (xy 80.01 64.77)
-		)
-		(stroke
-			(width 0)
-			(type default)
-		)
-	)
-	(wire
-		(pts
-			(xy 113.03 74.93) (xy 119.38 74.93)
-		)
-		(stroke
-			(width 0)
-			(type default)
-		)
-	)
-	(wire
-		(pts
-			(xy 113.03 77.47) (xy 119.38 77.47)
-		)
-		(stroke
-			(width 0)
-			(type default)
-		)
-	)
-	(wire
-		(pts
-			(xy 73.66 67.31) (xy 80.01 67.31)
+			(xy 157.48 64.77) (xy 163.83 64.77)
+		)
+		(stroke
+			(width 0)
+			(type default)
+		)
+	)
+	(wire
+		(pts
+			(xy 157.48 80.01) (xy 163.83 80.01)
+		)
+		(stroke
+			(width 0)
+			(type default)
+		)
+	)
+	(wire
+		(pts
+			(xy 157.48 69.85) (xy 163.83 69.85)
+		)
+		(stroke
+			(width 0)
+			(type default)
+		)
+	)
+	(wire
+		(pts
+			(xy 157.48 67.31) (xy 163.83 67.31)
+		)
+		(stroke
+			(width 0)
+			(type default)
+		)
+	)
+	(wire
+		(pts
+			(xy 119.38 66.04) (xy 124.46 66.04)
+		)
+		(stroke
+			(width 0)
+			(type default)
+		)
+	)
+	(wire
+		(pts
+			(xy 157.48 74.93) (xy 163.83 74.93)
+		)
+		(stroke
+			(width 0)
+			(type default)
+		)
+	)
+	(wire
+		(pts
+			(xy 157.48 77.47) (xy 163.83 77.47)
+		)
+		(stroke
+			(width 0)
+			(type default)
+		)
+	)
+	(wire
+		(pts
+			(xy 73.66 63.5) (xy 81.28 63.5)
+		)
+		(stroke
+			(width 0)
+			(type default)
+		)
+	)
+	(wire
+		(pts
+			(xy 73.66 66.04) (xy 81.28 66.04)
+		)
+		(stroke
+			(width 0)
+			(type default)
+		)
+	)
+	(wire
+		(pts
+			(xy 119.38 63.5) (xy 124.46 63.5)
 		)
 		(stroke
@@
 	)
 	(sheet
-		(at 119.38 60.96)
+		(at 163.83 60.96)
 		(size 33.02 34.29)
 		(exclude_from_sim no)
@@
 		)
 		(property "Sheetname" "Interface"
-			(at 119.38 60.2484 0)
+			(at 163.83 60.2484 0)
 			(effects
 				(font
@@
 		)
 		(property "Sheetfile" "Interface.kicad_sch"
-			(at 119.38 95.8346 0)
+			(at 163.83 95.8346 0)
 			(effects
 				(font
@@
 		)
 		(pin "UART0_RX" output
-			(at 119.38 64.77 180)
+			(at 163.83 64.77 180)
 			(effects
 				(font
@@
 		)
 		(pin "GPIO6" bidirectional
-			(at 119.38 80.01 180)
+			(at 163.83 80.01 180)
 			(effects
 				(font
@@
 		)
 		(pin "UART1_RX" output
-			(at 119.38 74.93 180)
+			(at 163.83 74.93 180)
 			(effects
 				(font
@@
 		)
 		(pin "UART1_TX" input
-			(at 119.38 77.47 180)
+			(at 163.83 77.47 180)
 			(effects
 				(font
@@
 		)
 		(pin "GPIO14" bidirectional
-			(at 119.38 69.85 180)
+			(at 163.83 69.85 180)
 			(effects
 				(font
@@
 		)
 		(pin "UART0_TX" input
-			(at 119.38 67.31 180)
+			(at 163.83 67.31 180)
 			(effects
 				(font
@@
 			(color 0 0 0 0.0000)
 		)
-		(property "Sheetname" "USB Input Isolation"
+		(property "Sheetname" "USB Input Protection & Filter"
 			(at 38.1 60.2484 0)
 			(effects
@@
 			)
 		)
-		(property "Sheetfile" "USB_input_isolation.kicad_sch"
+		(property "Sheetfile" "USB_input_protection.kicad_sch"
 			(at 38.1 95.8346 0)
 			(effects
@@
 			)
 		)
-		(pin "USB_D-" bidirectional
-			(at 73.66 67.31 0)
-			(effects
-				(font
-					(size 1.27 1.27)
-				)
-				(justify right)
-			)
-		)
-		(pin "USB_D+" bidirectional
-			(at 73.66 64.77 0)
+		(pin "USB_HOST_D-" bidirectional
+			(at 73.66 66.04 0)
+			(effects
+				(font
+					(size 1.27 1.27)
+				)
+				(justify right)
+			)
+		)
+		(pin "USB_HOST_D+" bidirectional
+			(at 73.66 63.5 0)
 			(effects
 				(font
@@
 	)
 	(sheet
-		(at 80.01 60.96)
-		(size 33.02 34.29)
+		(at 81.28 60.96)
+		(size 38.1 35.56)
 		(exclude_from_sim no)
 		(in_bom yes)
@@
 			(color 0 0 0 0.0000)
 		)
+		(property "Sheetname" "Galvanic Isolation"
+			(at 81.28 60.2484 0)
+			(effects
+				(font
+					(size 1.27 1.27)
+				)
+				(justify left bottom)
+			)
+		)
+		(property "Sheetfile" "galvanic_isolation.kicad_sch"
+			(at 81.28 97.1046 0)
+			(effects
+				(font
+					(size 1.27 1.27)
+				)
+				(justify left top)
+			)
+		)
+		(pin "USB_HOST_D-" bidirectional
+			(at 81.28 66.04 180)
+			(effects
+				(font
+					(size 1.27 1.27)
+				)
+				(justify left)
+			)
+		)
+		(pin "USB_HOST_D+" bidirectional
+			(at 81.28 63.5 180)
+			(effects
+				(font
+					(size 1.27 1.27)
+				)
+				(justify left)
+			)
+		)
+		(pin "USB_D-" bidirectional
+			(at 119.38 66.04 0)
+			(effects
+				(font
+					(size 1.27 1.27)
+				)
+				(justify right)
+			)
+		)
+		(pin "USB_D+" bidirectional
+			(at 119.38 63.5 0)
+			(effects
+				(font
+					(size 1.27 1.27)
+				)
+				(justify right)
+			)
+		)
+		(instances
+			(project "isolated_rp2040_debugger"
+				(path "/accec76c-f5c4-4bf8-be45-530a8e5bdaad"
+					(page "5")
+				)
+			)
+		)
+	)
+	(sheet
+		(at 124.46 60.96)
+		(size 33.02 34.29)
+		(exclude_from_sim no)
+		(in_bom yes)
+		(on_board yes)
+		(dnp no)
+		(fields_autoplaced yes)
+		(stroke
+			(width 0.1524)
+			(type solid)
+		)
+		(fill
+			(color 0 0 0 0.0000)
+		)
 		(property "Sheetname" "RP2040"
-			(at 80.01 60.2484 0)
+			(at 124.46 60.2484 0)
 			(effects
 				(font
@@
 		)
 		(property "Sheetfile" "RP2040.kicad_sch"
-			(at 80.01 95.8346 0)
+			(at 124.46 95.8346 0)
 			(effects
 				(font
@@
 		)
 		(pin "USB_D+" bidirectional
-			(at 80.01 64.77 180)
+			(at 124.46 63.5 180)
 			(effects
 				(font
@@
 		)
 		(pin "UART0_RX" input
-			(at 113.03 64.77 0)
+			(at 157.48 64.77 0)
 			(effects
 				(font
@@
 		)
 		(pin "GPIO14" bidirectional
-			(at 113.03 69.85 0)
+			(at 157.48 69.85 0)
 			(effects
 				(font
@@
 		)
 		(pin "GPIO6" bidirectional
-			(at 113.03 80.01 0)
+			(at 157.48 80.01 0)
 			(effects
 				(font
@@
 		)
 		(pin "UART0_TX" output
-			(at 113.03 67.31 0)
+			(at 157.48 67.31 0)
 			(effects
 				(font
@@
 		)
 		(pin "USB_D-" bidirectional
-			(at 80.01 67.31 180)
+			(at 124.46 66.04 180)
 			(effects
 				(font
@@
 		)
 		(pin "UART1_RX" input
-			(at 113.03 74.93 0)
+			(at 157.48 74.93 0)
 			(effects
 				(font
@@
 		)
 		(pin "UART1_TX" output
-			(at 113.03 77.47 0)
-			(effects
-				(font
+			(at 157.48 77.47 0)
+			(effects
+				(font
+					(size 1.27 1.27)
+				)
+				(justify right)
+			)
+		)
+		(pin "TGT_RST" output
+			(at 157.48 82.55 0)
+			(effects
+				(font
